File: MazeRobot_v2.kicad_sch (KiCad schematic)
At the start: 13 parts, among them SW1 SW_SPST, U3 TB6612FNG

Commit message: Add files via upload
Parts:
- added C1, C3: 0.1u, Capacitor_SMD:C_0603_1608Metric, symbol Device:C_Small
- added C2, C4, C5: 10u, Capacitor_SMD:C_0805_2012Metric, symbol Device:C_Small
- BT1, BT2: footprint (none) -> Connector_JST:JST_PH_S2B-PH-SM4-TB_1x02-1MP_P2.00mm_Horizontal; LCSC (none) -> C160404
- L-Back1, L-Front1, R-Back1, R-Front1: footprint (none) -> Connector_PinHeader_2.54mm:PinHeader_1x02_P2.54mm_Vertical_SMD_Pin1Left
- SW1: footprint (none) -> Button_Switch_SMD:SW_SPDT_PCM12
- U1: footprint (none) -> Package_TO_SOT_SMD:TO-263-5_TabPin3; LCSC (none) -> C77830
- U2: footprint (none) -> RF_Module:ESP32-WROOM-32E; LCSC (none) -> C701342
- U3: LCSC (none) -> C10553
- U4, U5: footprint (none) -> Connector_JST:JST_PH_S4B-PH-SM4-TB_1x04-1MP_P2.00mm_Horizontal
- U6: footprint (none) -> Connector_JST:JST_PH_S7B-PH-SM4-TB_1x07-1MP_P2.00mm_Horizontal
Connections:
- net +3V3: now also C3.1
- net +5V: now also C1.1, C2.1, C5.1
- net +7V4: now also C4.1
- net GND: now also C1.2, C2.2, C3.2, C4.2, C5.2
Other:
- note added: "Maya Raafat 900201982"
